File: i5tracker.kicad_pcb (KiCad board)
At the start: 2 copper layers, 78.7 x 55.9 mm, 25 parts, among them J1 Conn_01x06, J2 Conn_01x04, SW1 SW_SPST, SW2 SW_Push, U1 TP4056_board, U2 L7833, U3 ESP-WROOM-02, U4 MPU6500_board

Commit message: Add files via upload
Other:
- board text removed: "Ms.Amu loves her stomach. He's so hungry that He's been using Neos Tummy Force and established. He seems to eat before going to bed at night."
Changed lines of the file:
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@@
     (effects (font (size 2.5 2.5) (thickness 0.4)))
-  )
-  (gr_text "Ms.Amu loves her\nstomach.\nHe's so hungry that\nHe's been using \nNeos Tummy Force\nand established.\nHe seems to eat\n\n\n\nbefore going to\nbed at night." (at 123.825 75.565 90) (layer "F.SilkS")
-    (effects (font (size 1 1) (thickness 0.2)))
   )
   (segment (start 186.675 81.9) (end 172.085 67.31) (width 0.5) (layer "F.Cu") (net 1))
